File: pcb/output/NanoSoul/NanoSoul.kicad_sch (KiCad schematic)
At the start: 0 parts

Commit message: pcb: schematic-parity 真零(零 ignore) + 重导 Gerber
DRC `--schematic-parity --severity-all` = 0 violation / 0 unconnected /
0 schematic-parity,62 项检查全置 error、零 ignore(旧版的 7 项 ignore 全部真修掉,
非关检查)。verify_board 65/65、布线 778 走线+60 过孔未动。

- 修通 circuit-synth 原理图连通性:它把一器件所有网名标签堆在 pin1 → KiCad 推断错网。
  按 .net 逐脚在真实连接点重放 global_label(fix_sch_labels),net_conflict 199→0;
  真 NC 脚在板上配同名 unconnected- 网对齐(assign_nc_nets)。
- 板 Value 回填真实值(顺修「板上 Value=封装名」的 BOM bug)、lib_id 去库前缀(fix_board_meta);
  原理图删 circuit-synth 私有字段/封装过滤器、补缺失 Value(fix_sch_fields);
  J2 attr→through_hole(USB-C 靠屏蔽脚 THT 安装,属实);4×M3 孔标 board_only。
- 唯一保留例外 = J2(USB-C)连接器内部 DRU(实测 0.10mm 铜/0.185mm 孔,JLC 可造;
  KiCad 官方 USB_C_Receptacle_HRO 封装内部孔距也仅 0.15mm → 换封装消不掉、
  改窄焊盘会伤实焊。限 J2 内部两两对象,不放宽对板上走线)。
- 重导 Gerber(9 层 Protel 扩展名 + Excellon 钻孔)+ BOM/CPL。
Changed lines of the file:
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@@
 	(sheet
 		(at 25.4 12.7)
-		(size 48.1 71.12)
+		(size 48.1 76.2)
 		(exclude_from_sim no)
 		(in_bom yes)
@@
 		)
 		(property "Sheetfile" "Power.kicad_sch"
-			(at 25.4 84.4046 0)
+			(at 25.4 89.4846 0)
 			(effects
 				(font
@@
 		)
 		(pin "GND" bidirectional
-			(at 72.23 15.24 0)
+			(at 72.23 15.24 0.0000)
 			(effects
 				(font
@@
 		)
 		(pin "MOT_ISENSE" bidirectional
-			(at 72.23 17.78 0)
+			(at 72.23 17.78 0.0000)
 			(effects
 				(font
@@
 		)
 		(pin "MOT_RTN" bidirectional
-			(at 72.23 20.32 0)
+			(at 72.23 20.32 0.0000)
 			(effects
 				(font
@@
 		)
 		(pin "VMOT_F" bidirectional
-			(at 72.23 22.86 0)
+			(at 72.23 22.86 0.0000)
 			(effects
 				(font
@@
 		)
 		(pin "VSYS" bidirectional
-			(at 72.23 25.4 0)
+			(at 72.23 25.4 0.0000)
 			(effects
 				(font
@@
 		(instances
 			(project "NanoSoul"
-				(path "/cc6d016d-315a-4023-b551-816edf85e992"
+				(path "/d7c6fcf2-f77c-4139-a92e-1e725da500d2"
 					(page "2")
 				)
@@
 		)
 		(pin "GND" bidirectional
-			(at 135.73 15.24 0)
+			(at 135.73 15.24 0.0000)
 			(effects
 				(font
@@
 		)
 		(pin "I2C1_SCL" bidirectional
-			(at 135.73 17.78 0)
+			(at 135.73 17.78 0.0000)
 			(effects
 				(font
@@
 		)
 		(pin "I2C1_SDA" bidirectional
-			(at 135.73 20.32 0)
+			(at 135.73 20.32 0.0000)
 			(effects
 				(font
@@
 		)
 		(pin "IMU_CS" bidirectional
-			(at 135.73 22.86 0)
+			(at 135.73 22.86 0.0000)
 			(effects
 				(font
@@
 		)
 		(pin "IMU_INT" bidirectional
-			(at 135.73 25.4 0)
+			(at 135.73 25.4 0.0000)
 			(effects
 				(font
@@
 		)
 		(pin "IMU_MISO" bidirectional
-			(at 135.73 27.94 0)
+			(at 135.73 27.94 0.0000)
 			(effects
 				(font
@@
 		)
 		(pin "IMU_MOSI" bidirectional
-			(at 135.73 30.48 0)
+			(at 135.73 30.48 0.0000)
 			(effects
 				(font
@@
 		)
 		(pin "IMU_SCLK" bidirectional
-			(at 135.73 33.02 0)
+			(at 135.73 33.02 0.0000)
 			(effects
 				(font
@@
 		)
 		(pin "M0_ENC_A" bidirectional
-			(at 135.73 35.56 0)
+			(at 135.73 35.56 0.0000)
 			(effects
 				(font
@@
 		)
 		(pin "M0_ENC_B" bidirectional
-			(at 135.73 38.1 0)
+			(at 135.73 38.1 0.0000)
 			(effects
 				(font
@@
 		)
 		(pin "M0_IN1" bidirectional
-			(at 135.73 40.64 0)
+			(at 135.73 40.64 0.0000)
 			(effects
 				(font
@@
 		)
 		(pin "M0_IN2" bidirectional
-			(at 135.73 43.18 0)
+			(at 135.73 43.18 0.0000)
 			(effects
 				(font
@@
 		)
 		(pin "M0_PWM" bidirectional
-			(at 135.73 45.72 0)
+			(at 135.73 45.72 0.0000)
 			(effects
 				(font
@@
 		)
 		(pin "M1_ENC_A" bidirectional
-			(at 135.73 48.26 0)
+			(at 135.73 48.26 0.0000)
 			(effects
 				(font
@@
 		)
 		(pin "M1_ENC_B" bidirectional
-			(at 135.73 50.8 0)
+			(at 135.73 50.8 0.0000)
 			(effects
 				(font
@@
 		)
 		(pin "M1_IN1" bidirectional
-			(at 135.73 53.34 0)
+			(at 135.73 53.34 0.0000)
 			(effects
 				(font
@@
 		)
 		(pin "M1_IN2" bidirectional
-			(at 135.73 55.88 0)
+			(at 135.73 55.88 0.0000)
 			(effects
 				(font
@@
 		)
 		(pin "M1_PWM" bidirectional
-			(at 135.73 58.42 0)
+			(at 135.73 58.42 0.0000)
 			(effects
 				(font
@@
 		)
 		(pin "M2_ENC_A" bidirectional
-			(at 135.73 60.96 0)
+			(at 135.73 60.96 0.0000)
 			(effects
 				(font
@@
 		)
 		(pin "M2_ENC_B" bidirectional
-			(at 135.73 63.5 0)
+			(at 135.73 63.5 0.0000)
 			(effects
 				(font
@@
 		)
 		(pin "M2_IN1" bidirectional
-			(at 135.73 66.04 0)
+			(at 135.73 66.04 0.0000)
 			(effects
 				(font
@@
 		)
 		(pin "M2_IN2" bidirectional
-			(at 135.73 68.58 0)
+			(at 135.73 68.58 0.0000)
 			(effects
 				(font
@@
 		)
 		(pin "M2_PWM" bidirectional
-			(at 135.73 71.12 0)
+			(at 135.73 71.12 0.0000)
 			(effects
 				(font
@@
 		)
 		(pin "MOTOR_STBY" bidirectional
-			(at 135.73 73.66 0)
+			(at 135.73 73.66 0.0000)
 			(effects
 				(font
@@
 		)
 		(pin "MOT_ISENSE" bidirectional
-			(at 135.73 76.2 0)
+			(at 135.73 76.2 0.0000)
 			(effects
 				(font
@@
 		)
 		(pin "V3V3" bidirectional
-			(at 135.73 78.74 0)
+			(at 135.73 78.74 0.0000)
 			(effects
 				(font
@@
 		)
 		(pin "VSYS" bidirectional
-			(at 135.73 81.28 0)
+			(at 135.73 81.28 0.0000)
 			(effects
 				(font
@@
 		(instances
 			(project "NanoSoul"
-				(path "/cc6d016d-315a-4023-b551-816edf85e992"
+				(path "/d7c6fcf2-f77c-4139-a92e-1e725da500d2"
 					(page "2")
 				)
@@
 		)
 		(pin "GND" bidirectional
-			(at 197.96 15.24 0)
+			(at 197.96 15.24 0.0000)
 			(effects
 				(font
@@
 		)
 		(pin "M0_ENC_A" bidirectional
-			(at 197.96 17.78 0)
+			(at 197.96 17.78 0.0000)
 			(effects
 				(font
@@
 		)
 		(pin "M0_ENC_B" bidirectional
-			(at 197.96 20.32 0)
+			(at 197.96 20.32 0.0000)
 			(effects
 				(font
@@
 		)
 		(pin "M0_IN1" bidirectional
-			(at 197.96 22.86 0)
+			(at 197.96 22.86 0.0000)
 			(effects
 				(font
@@
 		)
 		(pin "M0_IN2" bidirectional
-			(at 197.96 25.4 0)
+			(at 197.96 25.4 0.0000)
 			(effects
 				(font
@@
 		)
 		(pin "M0_PWM" bidirectional
-			(at 197.96 27.94 0)
+			(at 197.96 27.94 0.0000)
 			(effects
 				(font
@@
 		)
 		(pin "M1_ENC_A" bidirectional
-			(at 197.96 30.48 0)
+			(at 197.96 30.48 0.0000)
 			(effects
 				(font
@@
 		)
 		(pin "M1_ENC_B" bidirectional
-			(at 197.96 33.02 0)
+			(at 197.96 33.02 0.0000)
 			(effects
 				(font
@@
 		)
 		(pin "M1_IN1" bidirectional
-			(at 197.96 35.56 0)
+			(at 197.96 35.56 0.0000)
 			(effects
 				(font
@@
 		)
 		(pin "M1_IN2" bidirectional
-			(at 197.96 38.1 0)
+			(at 197.96 38.1 0.0000)
 			(effects
 				(font
@@
 		)
 		(pin "M1_PWM" bidirectional
-			(at 197.96 40.64 0)
+			(at 197.96 40.64 0.0000)
 			(effects
 				(font
@@
 		)
 		(pin "M2_ENC_A" bidirectional
-			(at 197.96 43.18 0)
+			(at 197.96 43.18 0.0000)
 			(effects
 				(font
@@
 		)
 		(pin "M2_ENC_B" bidirectional
-			(at 197.96 45.72 0)
+			(at 197.96 45.72 0.0000)
 			(effects
 				(font
@@
 		)
 		(pin "M2_IN1" bidirectional
-			(at 197.96 48.26 0)
+			(at 197.96 48.26 0.0000)
 			(effects
 				(font
@@
 		)
 		(pin "M2_IN2" bidirectional
-			(at 197.96 50.8 0)
+			(at 197.96 50.8 0.0000)
 			(effects
 				(font
@@
 		)
 		(pin "M2_PWM" bidirectional
-			(at 197.96 53.34 0)
+			(at 197.96 53.34 0.0000)
 			(effects
 				(font
@@
 		)
 		(pin "MOTOR_STBY" bidirectional
-			(at 197.96 55.88 0)
+			(at 197.96 55.88 0.0000)
 			(effects
 				(font
@@
 		)
 		(pin "MOT_RTN" bidirectional
-			(at 197.96 58.42 0)
+			(at 197.96 58.42 0.0000)
 			(effects
 				(font
@@
 		)
 		(pin "V3V3" bidirectional
-			(at 197.96 60.96 0)
+			(at 197.96 60.96 0.0000)
 			(effects
 				(font
@@
 		)
 		(pin "VMOT_F" bidirectional
-			(at 197.96 63.5 0)
+			(at 197.96 63.5 0.0000)
 			(effects
 				(font
@@
 		(instances
 			(project "NanoSoul"
-				(path "/cc6d016d-315a-4023-b551-816edf85e992"
+				(path "/d7c6fcf2-f77c-4139-a92e-1e725da500d2"
 					(page "2")
 				)
@@
 		)
 		(pin "GND" bidirectional
-			(at 258.92 15.24 0)
+			(at 258.92 15.24 0.0000)
 			(effects
 				(font
@@
 		)
 		(pin "I2C1_SCL" bidirectional
-			(at 258.92 17.78 0)
+			(at 258.92 17.78 0.0000)
 			(effects
 				(font
@@
 		)
 		(pin "I2C1_SDA" bidirectional
-			(at 258.92 20.32 0)
+			(at 258.92 20.32 0.0000)
 			(effects
 				(font
@@
 		)
 		(pin "IMU_CS" bidirectional
-			(at 258.92 22.86 0)
+			(at 258.92 22.86 0.0000)
 			(effects
 				(font
@@
 		)
 		(pin "IMU_INT" bidirectional
-			(at 258.92 25.4 0)
+			(at 258.92 25.4 0.0000)
 			(effects
 				(font
@@
 		)
 		(pin "IMU_MISO" bidirectional
-			(at 258.92 27.94 0)
+			(at 258.92 27.94 0.0000)
 			(effects
 				(font
@@
 		)
 		(pin "IMU_MOSI" bidirectional
-			(at 258.92 30.48 0)
+			(at 258.92 30.48 0.0000)
 			(effects
 				(font
@@
 		)
 		(pin "IMU_SCLK" bidirectional
-			(at 258.92 33.02 0)
+			(at 258.92 33.02 0.0000)
 			(effects
 				(font
@@
 		)
 		(pin "V3V3" bidirectional
-			(at 258.92 35.56 0)
+			(at 258.92 35.56 0.0000)
 			(effects
 				(font
@@
 		(instances
 			(project "NanoSoul"
-				(path "/cc6d016d-315a-4023-b551-816edf85e992"
+				(path "/d7c6fcf2-f77c-4139-a92e-1e725da500d2"
 					(page "2")
 				)
