File: pcb/output/NanoSoul/Power.kicad_sch (KiCad schematic)
At the start: 32 parts

Commit message: pcb: 3mm 白边 + J2/J7 离 J4 + DRC 丝印告警清零
- 最外围 3mm 白边：板放大到 94×92（Ø108 切边收小到 7/8mm），铜/器件焊盘距最外缘 ≥3mm
  （自动布线内缩 3mm；顶排 J5/J6 下移、J8 左移退出白边区）。
- J2/J7 离 J4：右月牙整体右移 1.6mm，离 J4 本体 +0.83mm（原相擦 0.78mm）。
- DRC = 0 warning：5 个位号(D4/D5/Q1/U1/U7)挪开、接线图例升到 0.8mm 并缩短、
  删 J3/J4 压挖孔丝印、隐藏 6 安装孔与 U7 位号。
- 17.8mm 母座行距核对通过；4 个 M3 安装孔成规则 54×82 矩形（旧版钉在 Ø108 圆外、钻不出，已修正）。
- 余 MOT_RTN/GND 各 1 段跨挖孔大电流网/地：按 docs 铁律出板前人工绕挖孔补（GND 建议铺地铜），
  网表连接关系正确（其余 170 网 0 短路）。原理图 ERC 不适用：circuit-synth 开源导出无导线、
  网表为真值源。详见 docs/05 §9.1。
Parts:
- C1, C2, C3, C4, C5, C6, C7, C8, C9, D1, D2, D3, D4, D5, F1, J1, J2, Q1, R1, R2, R3, R4, R5, R6, R7, R8, SW1, U1, U2, U3: hierarchy_path /8a83f0c7-8320-4874-8ea1-ef8ee28a330a/d7f127d6-54c6-42d2-b6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 -> /cc6d016d-315a-4023-b551-816edf85e992/02c281f0-3e36-4ec8-b2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; root_uuid 8a83f0c7-8320-4874-8ea1-ef8ee28a330a -> cc6d016d-315a-4023-b551-816edf85e992
- L1, L2: footprint Inductor_SMD:L_12x12mm_H8mm -> Inductor_SMD:L_6.3x6.3_H3; hierarchy_path /8a83f0c7-8320-4874-8ea1-ef8ee28a330a/d7f127d6-54c6-42d2-b6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 -> /cc6d016d-315a-4023-b551-816edf85e992/02c281f0-3e36-4ec8-b2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; root_uuid 8a83f0c7-8320-4874-8ea1-ef8ee28a330a -> cc6d016d-315a-4023-b551-816edf85e992

Commit message: pcb: schematic-parity 真零(零 ignore) + 重导 Gerber
DRC `--schematic-parity --severity-all` = 0 violation / 0 unconnected /
0 schematic-parity,62 项检查全置 error、零 ignore(旧版的 7 项 ignore 全部真修掉,
非关检查)。verify_board 65/65、布线 778 走线+60 过孔未动。

- 修通 circuit-synth 原理图连通性:它把一器件所有网名标签堆在 pin1 → KiCad 推断错网。
  按 .net 逐脚在真实连接点重放 global_label(fix_sch_labels),net_conflict 199→0;
  真 NC 脚在板上配同名 unconnected- 网对齐(assign_nc_nets)。
- 板 Value 回填真实值(顺修「板上 Value=封装名」的 BOM bug)、lib_id 去库前缀(fix_board_meta);
  原理图删 circuit-synth 私有字段/封装过滤器、补缺失 Value(fix_sch_fields);
  J2 attr→through_hole(USB-C 靠屏蔽脚 THT 安装,属实);4×M3 孔标 board_only。
- 唯一保留例外 = J2(USB-C)连接器内部 DRU(实测 0.10mm 铜/0.185mm 孔,JLC 可造;
  KiCad 官方 USB_C_Receptacle_HRO 封装内部孔距也仅 0.15mm → 换封装消不掉、
  改窄焊盘会伤实焊。限 J2 内部两两对象,不放宽对板上走线)。
- 重导 Gerber(9 层 Protel 扩展名 + Excellon 钻孔)+ BOM/CPL。
Parts:
- removed J2: (no value), Connector_PinHeader_2.54mm:PinHeader_1x02_P2.54mm_Vertical, symbol Connector_Generic:Conn_01x02
- added J2: USB-C_SMD-TYPE-C-31-M-12_1, USB-C_SMD-TYPE-C-31-M-12_1, symbol nanosoul:TYPE-C-31-M-12
- added R10: 1k, R_0603_1608Metric, symbol Device:R
- added R9: 0.05, R_0805_2012Metric, symbol Device:R
- C1, C4, C9: footprint Capacitor_SMD:C_0603_1608Metric -> C_0603_1608Metric; hierarchy_path /cc6d016d-315a-4023-b551-816edf85e992/02c281f0-3e36-4ec8-b2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 -> (none); project_name NanoSoul -> (none); root_uuid cc6d016d-315a-4023-b551-816edf85e992 -> (none)
- C2, C3, C5, C6, C7: footprint Capacitor_SMD:C_0805_2012Metric -> C_0805_2012Metric; hierarchy_path /cc6d016d-315a-4023-b551-816edf85e992/02c281f0-3e36-4ec8-b2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 -> (none); project_name NanoSoul -> (none); root_uuid cc6d016d-315a-4023-b551-816edf85e992 -> (none)
- C8: footprint Capacitor_SMD:CP_Elec_8x10.5 -> CP_Elec_8x10.5; hierarchy_path /cc6d016d-315a-4023-b551-816edf85e992/02c281f0-3e36-4ec8-b2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 -> (none); project_name NanoSoul -> (none); root_uuid cc6d016d-315a-4023-b551-816edf85e992 -> (none)
- D1, D2, D3: value (none) -> LED_0805_2012Metric; footprint LED_SMD:LED_0805_2012Metric -> LED_0805_2012Metric; hierarchy_path /cc6d016d-315a-4023-b551-816edf85e992/02c281f0-3e36-4ec8-b2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 -> (none); project_name NanoSoul -> (none); root_uuid cc6d016d-315a-4023-b551-816edf85e992 -> (none)
- D4, D5: value (none) -> SMA_L4.3-W2.7-LS5.1-RD; footprint nanosoul:SMA_L4.3-W2.7-LS5.1-RD -> SMA_L4.3-W2.7-LS5.1-RD; hierarchy_path /cc6d016d-315a-4023-b551-816edf85e992/02c281f0-3e36-4ec8-b2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 -> (none); project_name NanoSoul -> (none); root_uuid cc6d016d-315a-4023-b551-816edf85e992 -> (none)
- F1: footprint Fuse:Fuse_0805_2012Metric -> Fuse_0805_2012Metric; hierarchy_path /cc6d016d-315a-4023-b551-816edf85e992/02c281f0-3e36-4ec8-b2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 -> (none); project_name NanoSoul -> (none); root_uuid cc6d016d-315a-4023-b551-816edf85e992 -> (none)
- J1: value (none) -> JST_PH_B2B-PH-K_1x02_P2.00mm_Vertical; footprint Connector_JST:JST_PH_B2B-PH-K_1x02_P2.00mm_Vertical -> JST_PH_B2B-PH-K_1x02_P2.00mm_Vertical; hierarchy_path /cc6d016d-315a-4023-b551-816edf85e992/02c281f0-3e36-4ec8-b2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 -> (none); project_name NanoSoul -> (none); root_uuid cc6d016d-315a-4023-b551-816edf85e992 -> (none)
- L1, L2: footprint Inductor_SMD:L_6.3x6.3_H3 -> L_6.3x6.3_H3; hierarchy_path /cc6d016d-315a-4023-b551-816edf85e992/02c281f0-3e36-4ec8-b2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 -> (none); project_name NanoSoul -> (none); root_uuid cc6d016d-315a-4023-b551-816edf85e992 -> (none)
- Q1: value (none) -> SOT-23-6_L2.9-W1.6-P0.95-LS2.8-BR; footprint nanosoul:SOT-23-6_L2.9-W1.6-P0.95-LS2.8-BR -> SOT-23-6_L2.9-W1.6-P0.95-LS2.8-BR; hierarchy_path /cc6d016d-315a-4023-b551-816edf85e992/02c281f0-3e36-4ec8-b2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 -> (none); project_name NanoSoul -> (none); root_uuid cc6d016d-315a-4023-b551-816edf85e992 -> (none)
- R1, R2, R3, R4: footprint Resistor_SMD:R_0603_1608Metric -> R_0603_1608Metric; hierarchy_path /cc6d016d-315a-4023-b551-816edf85e992/02c281f0-3e36-4ec8-b2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 -> (none); project_name NanoSoul -> (none); root_uuid cc6d016d-315a-4023-b551-816edf85e992 -> (none)
- R5: value 91k -> 5.1k; footprint Resistor_SMD:R_0603_1608Metric -> R_0603_1608Metric; hierarchy_path /cc6d016d-315a-4023-b551-816edf85e992/02c281f0-3e36-4ec8-b2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 -> (none); project_name NanoSoul -> (none); root_uuid cc6d016d-315a-4023-b551-816edf85e992 -> (none)
- R6: value 10k -> 5.1k; footprint Resistor_SMD:R_0603_1608Metric -> R_0603_1608Metric; hierarchy_path /cc6d016d-315a-4023-b551-816edf85e992/02c281f0-3e36-4ec8-b2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 -> (none); project_name NanoSoul -> (none); root_uuid cc6d016d-315a-4023-b551-816edf85e992 -> (none)
- R7: value 0.05 -> 82k; footprint Resistor_SMD:R_0805_2012Metric -> R_0603_1608Metric; hierarchy_path /cc6d016d-315a-4023-b551-816edf85e992/02c281f0-3e36-4ec8-b2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 -> (none); project_name NanoSoul -> (none); root_uuid cc6d016d-315a-4023-b551-816edf85e992 -> (none)
- R8: value 1k -> 10k; footprint Resistor_SMD:R_0603_1608Metric -> R_0603_1608Metric; hierarchy_path /cc6d016d-315a-4023-b551-816edf85e992/02c281f0-3e36-4ec8-b2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 -> (none); project_name NanoSoul -> (none); root_uuid cc6d016d-315a-4023-b551-816edf85e992 -> (none)
- SW1: value (none) -> SW_SPST_CK_RS282G05A3; footprint Button_Switch_SMD:SW_SPST_CK_RS282G05A3 -> SW_SPST_CK_RS282G05A3; hierarchy_path /cc6d016d-315a-4023-b551-816edf85e992/02c281f0-3e36-4ec8-b2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 -> (none); project_name NanoSoul -> (none); root_uuid cc6d016d-315a-4023-b551-816edf85e992 -> (none)
- U1, U3: value (none) -> SOT-23-6_L2.9-W1.6-P0.95-LS2.8-BL; footprint nanosoul:SOT-23-6_L2.9-W1.6-P0.95-LS2.8-BL -> SOT-23-6_L2.9-W1.6-P0.95-LS2.8-BL; hierarchy_path /cc6d016d-315a-4023-b551-816edf85e992/02c281f0-3e36-4ec8-b2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 -> (none); project_name NanoSoul -> (none); root_uuid cc6d016d-315a-4023-b551-816edf85e992 -> (none)
- U2: value (none) -> ESOP-8_L4.9-W3.9-P1.27-LS6.0-BL-EP2.0; footprint nanosoul:ESOP-8_L4.9-W3.9-P1.27-LS6.0-BL-EP2.0 -> ESOP-8_L4.9-W3.9-P1.27-LS6.0-BL-EP2.0; hierarchy_path /cc6d016d-315a-4023-b551-816edf85e992/02c281f0-3e36-4ec8-b2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 -> (none); project_name NanoSoul -> (none); root_uuid cc6d016d-315a-4023-b551-816edf85e992 -> (none)
Connections:
- net CELL_MINUS: now also C1.2; no longer C1.1, R1.1, U1.5 (VCC)
- net CHG_IN: now also J2.A4B9 (VBUS), J2.B4A9 (VBUS); no longer C2.1, C3.1, C4.1, C6.1, C7.1, C8.1, C9.1, D1.2 (A), D2.2 (A), D3.2 (A), D4.1 (C), D5.2 (A), F1.1, Q1.3 (S2), R2.1, R3.1, R4.1, R5.1, R6.1, R7.1, R8.1, SW1.2, U1.2 (VM), U2.8 (VOUT), U2.9 (EP), U3.2 (GND), U3.3 (FB)
- net DRAIN_COM: now also Q1.5 (D1/D2)
- net LED_A2: now reaches R3.2
- net LED_A2: now also D2.2 (A)
- net GND: now reaches C9.2
- net GND: now also C2.2, C3.2, C4.2, C5.2, C6.2, C7.2, C8.2, Q1.3 (S2), R5.2, R6.2, R8.2, SW1.2, U1.2 (VM), U2.9 (EP), U3.2 (GND), J2.1 (EH), J2.2 (EH), J2.3 (EH), J2.4 (EH), J2.A1B12 (GND), J2.B1A12 (GND), R9.2
- net VMOT_F: now reaches F1.2
- net VMOT_F: now also C8.1
- net VBAT: now reaches J1.1 (Pin_1)
- net VBAT: now also C2.1, C6.1, L1.1, L2.1, R1.1, U2.6 (BAT), U3.4 (EN), U3.5 (IN)
- net LED_A3: now reaches R4.2
- net LED_A3: now also D3.2 (A)
- net DW_VCC: now reaches R1.2
- net DW_VCC: now also C1.1, U1.5 (VCC)
- net LED_A1: now reaches R2.2
- net LED_A1: now also D1.2 (A)
- net MT_FB: now reaches R7.2
- net MT_FB: now also R8.1, U3.3 (FB)
- new net MOT_ISENSE: C9.1, R10.2
- new net MOT_RTN: R10.1, R9.1
- new net USB_CC1: J2.A5 (CC1), R5.1
- new net USB_CC2: J2.B5 (CC2), R6.1
- new net V5: C3.1, C4.1, D5.2 (A), R2.1, R3.1, R4.1, U2.8 (VOUT)
- new net VMOT: C7.1, D4.1 (C), F1.1, R7.1

Commit message: pcb: 修嘉立创 SMT 单两处"邮寄/停产"料 — U6→QMI8658A、R9 shunt→1206
SMT 下单核对单 待邮寄(2): U6 IMU 停产、R9 shunt 无现货。改为全现货可自动贴装：

- U6 IMU: QMI8658C(C2842151,JLC SMT 停产/邮寄) → 同族 QMI8658A(C3021082,
  现货 39k)。同 LGA-14、4 线 SPI 脚位完全一致(A 版 datasheet 13-52-25
  Table3+Fig4 逐脚核过:1=SDO/4=INT1/5=VDDIO/6,7=GND/8=VDD/12=CS/13=SCL/
  14=SDA,2/3/9/10/11 SPI 下可悬空)、驱动同(SensorLib/Waveshare)→ 板/固件不动,仅换料号。
- R9 50mΩ 电流采样 shunt: 0805 50mΩ 在 JLC 无现货(UNI-ROYAL C127697 仅 4 颗、
  Yageo 0805 R05L 不在库) → 改 1206 Yageo RL1206FR-070R05L(C375525,现货 15k/250mW/
  AEC-Q200)。板上【原地换封装】(焊盘 1.125×1.75、丝印/courtyard/fab 几何全取官方
  R_1206_3216Metric)，阻值 50mΩ 不变、位置/网络不变;开放区无邻件、走线仍连通。
- DRC --schematic-parity --severity-all = 0/0/0、parity 0、verify_board 65/65 不变。
- 重导 Gerber(9 层 Protel)+ BOM/CPL;BOM 30 行全带 LCSC、全现货(无留空/邮寄/停产)。
Parts:
- R9: footprint R_0805_2012Metric -> R_1206_3216Metric
Changed lines of the file:
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@@
 			)
 		)
-		(property "Footprint" "R_0805_2012Metric"
+		(property "Footprint" "R_1206_3216Metric"
 			(at 252.222 104.14 90)
 			(effects
