File: pcb/output/NanoSoul/Power.kicad_sch (KiCad schematic)
At the start: 34 parts, among them J1 JST_PH_B2B-PH-K_1x02_P2.00mm_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, J2 USB-C_SMD-TYPE-C-31-M-12_1, Q1 SOT-23-6_L2.9-W1.6-P0.95-LS2.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, SW1 SW_SPST_CK_RS282G05A3, U1 SOT-23-6_L2.9-W1.6-P0.95-LS2.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, U2 ESOP-8_L4.9-W3.9-P1.27-LS6.0-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, U3 SOT-23-6_L2.9-W1.6-P0.95-LS2.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

Commit message: pcb: 修嘉立创 SMT 三处封装-实物不符(SW1/R9/L1/L2) — 混合改法, DRC/ERC 0
JLC PCBA DFM 三条(对提交板 94×92):
- SW1 器件选小: 封装是 C&K RS-282 宽盘、配的却是小的 TS-1088 → 改板:焊盘收到
  C720477 官方 land(±2.18,1.23×1.86)+重布 KEY_BTN/GND 两脚。保留便宜的 TS-1088(C720477)。
- R9 器件选大/不匹配: R_1206 盘配 C375525(Yageo,盘略大) → 改板:焊盘放大到 C375525
  官方 land(±1.48,1.208×1.701)。保留在库件 C375525(50mΩ shunt)。
- L1/L2 引脚类型/焊盘不符(偏位虚焊): 通用小盘(1.5×2.4)对不上 6.3×6.3 电感端子 →
  换料+改盘:换库存足的 Sunlord SWPA6045(替代库存薄的 LQH66S),焊盘放大到其官方 land
  (2.474×5.020@±2.60)+VBAT 让位重布。L2=SWPA6045S4R7MT(C78804,4.7µH/3.6A);
  L1=SWPA6045S2R2NT(2.2µH/5A,同 land)— 其 JLC C 号请下单页按型号确认(本机环境拉不到)。

- lib_id 保留原名(SW-SMD/R_1206/L_6.3x6.3)对齐原理图 → schematic-parity 0。
- 复核:DRC 0 违规/0 未连/parity 0、ERC 0;重导 9 层 Protel Gerber + BOM/CPL。
Parts:
- SW1: footprint SW_SPST_CK_RS282G05A3 -> SW-SMD_L3.9-W3.0-P4.45
Changed lines of the file:
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@@
 			)
 		)
-		(property "Footprint" "SW_SPST_CK_RS282G05A3"
+		(property "Footprint" "SW-SMD_L3.9-W3.0-P4.45"
 			(at 266.7 30.48 0.0000)
 			(effects
